File: shrug75/shrug75.kicad_pcb (KiCad board)
At the start: 2 copper layers, 303.8 x 115.3 mm, 0 parts

Commit message: Placing the switches
Parts:
- added A1: MX-NoLED, MX_Only:MXOnly-1U-NoLED, F.Cu at (105.9, 155.6)
- added APOS1: MX-NoLED, MX_Only:MXOnly-1U-NoLED, F.Cu at (296.3, 155.6)
- added B1: MX-NoLED, MX_Only:MXOnly-1U-NoLED, F.Cu at (191.6, 174.7)
- added BACKSLASH1: MX-NoLED, MX_Only:MXOnly-1U-NoLED, F.Cu at (334.5, 136.6)
- added BACKSPACE1: MX-NoLED, MX_Only:MXOnly-2U-NoLED, F.Cu at (329.7, 117.5)
- added BACKTICK1: MX-NoLED, MX_Only:MXOnly-1U-NoLED, F.Cu at (72.5, 117.5)
- added C1: 0.1uF, Capacitor_SMD:C_0805_2012Metric, F.Cu at (318.4, 293.0)
- added C10: 0.1uF, Capacitor_SMD:C_0805_2012Metric, F.Cu at (318.4, 286.9)
- added C2: 22pF, Capacitor_SMD:C_0805_2012Metric, F.Cu at (327.3, 289.9)
- added C3: 22pF, Capacitor_SMD:C_0805_2012Metric, F.Cu at (352.1, 263.7)
- added C4: 0.1uF, Capacitor_SMD:C_0805_2012Metric, F.Cu at (327.3, 286.9)
- added C5: 0.1uF, Capacitor_SMD:C_0805_2012Metric, F.Cu at (331.8, 283.9)
- added C6: 0.1uF, Capacitor_SMD:C_0805_2012Metric, F.Cu at (327.3, 283.9)
- added C8: 1uF, Capacitor_SMD:C_0805_2012Metric, F.Cu at (322.9, 293.0)
- added C9: 0.1uF, Capacitor_SMD:C_0805_2012Metric, F.Cu at (314.0, 290.0)
- added CAPSLOCK1: MX-LED, MX_Only:MXOnly-1U-NoLED, F.Cu at (79.7, 155.6)
- added COMA1: MX-NoLED, MX_Only:MXOnly-1U-NoLED, F.Cu at (248.7, 174.7)
- added C_KEY1: MX-NoLED, MX_Only:MXOnly-1U-NoLED, F.Cu at (153.5, 174.7)
- added D1: D_Small, Diode_SMD:D_0805_2012Metric, F.Cu at (302.7, 304.1)
- added D10: D_Small, Diode_SMD:D_0805_2012Metric, F.Cu at (131.0, 381.2)
- added D11: D_Small, Diode_SMD:D_0805_2012Metric, F.Cu at (352.3, 229.4)
- added D12: D_Small, Diode_SMD:D_0805_2012Metric, F.Cu at (352.3, 226.3)
- added D13: D_Small, Diode_SMD:D_0805_2012Metric, F.Cu at (352.3, 223.3)
- added D14: D_Small, Diode_SMD:D_0805_2012Metric, F.Cu at (144.4, 381.2)
- added D15: D_Small, Diode_SMD:D_0805_2012Metric, F.Cu at (139.9, 381.2)
- added D16: D_Small, Diode_SMD:D_0805_2012Metric, F.Cu at (144.4, 378.1)
- added D17: D_Small, Diode_SMD:D_0805_2012Metric, F.Cu at (139.9, 378.1)
- added D18: D_Small, Diode_SMD:D_0805_2012Metric, F.Cu at (352.3, 244.6)
- added D19: D_Small, Diode_SMD:D_0805_2012Metric, F.Cu at (144.4, 372.1)
- added D2: D_Small, Diode_SMD:D_0805_2012Metric, F.Cu at (293.8, 310.2)
- added D20: D_Small, Diode_SMD:D_0805_2012Metric, F.Cu at (139.9, 375.1)
- added D21: D_Small, Diode_SMD:D_0805_2012Metric, F.Cu at (135.5, 381.2)
- added D22: D_Small, Diode_SMD:D_0805_2012Metric, F.Cu at (352.3, 232.4)
- added D23: D_Small, Diode_SMD:D_0805_2012Metric, F.Cu at (352.3, 259.8)
- added D24: D_Small, Diode_SMD:D_0805_2012Metric, F.Cu at (352.3, 256.7)
- added D25: D_Small, Diode_SMD:D_0805_2012Metric, F.Cu at (314.0, 302.1)
- added D27: D_Small, Diode_SMD:D_0805_2012Metric, F.Cu at (318.5, 299.0)
- added D28: D_Small, Diode_SMD:D_0805_2012Metric, F.Cu at (314.0, 299.0)
- added D29: D_Small, Diode_SMD:D_0805_2012Metric, F.Cu at (318.5, 296.0)
- added D3: D_Small, Diode_SMD:D_0805_2012Metric, F.Cu at (298.3, 307.1)
- added D30: D_Small, Diode_SMD:D_0805_2012Metric, F.Cu at (314.0, 296.0)
- added D31: D_Small, Diode_SMD:D_0805_2012Metric, F.Cu at (322.9, 283.9)
- added D32: D_Small, Diode_SMD:D_0805_2012Metric, F.Cu at (122.1, 378.1)
- added D33: D_Small, Diode_SMD:D_0805_2012Metric, F.Cu at (135.5, 375.1)
- added D34: D_Small, Diode_SMD:D_0805_2012Metric, F.Cu at (131.0, 375.1)
- added D35: D_Small, Diode_SMD:D_0805_2012Metric, F.Cu at (126.6, 375.1)
- added D36: D_Small, Diode_SMD:D_0805_2012Metric, F.Cu at (113.2, 377.1)
- added D37: D_Small, Diode_SMD:D_0805_2012Metric, F.Cu at (139.9, 372.1)
- added D38: D_Small, Diode_SMD:D_0805_2012Metric, F.Cu at (135.5, 372.1)
- added D39: D_Small, Diode_SMD:D_0805_2012Metric, F.Cu at (225.2, 270.0)
- added D4: D_Small, Diode_SMD:D_0805_2012Metric, F.Cu at (352.3, 250.7)
- added D40: D_Small, Diode_SMD:D_0805_2012Metric, F.Cu at (126.6, 372.1)
- added D41: D_Small, Diode_SMD:D_0805_2012Metric, F.Cu at (144.4, 369.0)
- added D42: D_Small, Diode_SMD:D_0805_2012Metric, F.Cu at (139.9, 369.0)
- added D43: D_Small, Diode_SMD:D_0805_2012Metric, F.Cu at (126.6, 378.1)
- added D44: D_Small, Diode_SMD:D_0805_2012Metric, F.Cu at (135.5, 369.0)
- added D45: D_Small, Diode_SMD:D_0805_2012Metric, F.Cu at (131.0, 369.0)
- added D46: D_Small, Diode_SMD:D_0805_2012Metric, F.Cu at (144.4, 366.0)
- added D47: D_Small, Diode_SMD:D_0805_2012Metric, F.Cu at (139.9, 366.0)
- added D48: D_Small, Diode_SMD:D_0805_2012Metric, F.Cu at (225.2, 273.0)
- added D49: D_Small, Diode_SMD:D_0805_2012Metric, F.Cu at (225.2, 276.0)
- added D5: D_Small, Diode_SMD:D_0805_2012Metric, F.Cu at (322.9, 289.9)
- added D50: D_Small, Diode_SMD:D_0805_2012Metric, F.Cu at (220.8, 279.1)
- added D51: D_Small, Diode_SMD:D_0805_2012Metric, F.Cu at (225.2, 279.1)
- added D52: D_Small, Diode_SMD:D_0805_2012Metric, F.Cu at (135.5, 366.0)
- added D53: D_Small, Diode_SMD:D_0805_2012Metric, F.Cu at (108.8, 380.1)
- added D54: D_Small, Diode_SMD:D_0805_2012Metric, F.Cu at (77.1, 381.9)
- added D55: D_Small, Diode_SMD:D_0805_2012Metric, F.Cu at (131.0, 366.0)
- added D56: D_Small, Diode_SMD:D_0805_2012Metric, F.Cu at (126.6, 369.0)
- added D57: D_Small, Diode_SMD:D_0805_2012Metric, F.Cu at (122.1, 375.1)
- added D58: D_Small, Diode_SMD:D_0805_2012Metric, F.Cu at (117.7, 377.7)
- added D59: D_Small, Diode_SMD:D_0805_2012Metric, F.Cu at (113.2, 380.1)
- added D6: D_Small, Diode_SMD:D_0805_2012Metric, F.Cu at (144.4, 375.1)
- added D60: D_Small, Diode_SMD:D_0805_2012Metric, F.Cu at (117.7, 374.6)
- added D61: D_Small, Diode_SMD:D_0805_2012Metric, F.Cu at (122.1, 372.1)
- added D62: D_Small, Diode_SMD:D_0805_2012Metric, F.Cu at (122.1, 369.0)
- added D63: D_Small, Diode_SMD:D_0805_2012Metric, F.Cu at (126.6, 366.0)
- added D64: D_Small, Diode_SMD:D_0805_2012Metric, F.Cu at (122.1, 366.0)
- added D65: D_Small, Diode_SMD:D_0805_2012Metric, F.Cu at (117.7, 371.6)
- added D66: D_Small, Diode_SMD:D_0805_2012Metric, F.Cu at (220.8, 275.6)
- added D67: D_Small, Diode_SMD:D_0805_2012Metric, F.Cu at (81.5, 381.9)
- added D68: D_Small, Diode_SMD:D_0805_2012Metric, F.Cu at (99.9, 381.1)
- added D69: D_Small, Diode_SMD:D_0805_2012Metric, F.Cu at (104.3, 381.1)
- added D7: D_Small, Diode_SMD:D_0805_2012Metric, F.Cu at (352.3, 241.5)
- added D70: D_Small, Diode_SMD:D_0805_2012Metric, F.Cu at (108.8, 377.1)
- added D71: D_Small, Diode_SMD:D_0805_2012Metric, F.Cu at (95.4, 381.1)
- added D72: D_Small, Diode_SMD:D_0805_2012Metric, F.Cu at (131.0, 372.1)
- added D73: D_Small, Diode_SMD:D_0805_2012Metric, F.Cu at (126.6, 381.2)
- added D74: D_Small, Diode_SMD:D_0805_2012Metric, F.Cu at (122.1, 381.2)
- added D75: D_Small, Diode_SMD:D_0805_2012Metric, F.Cu at (117.7, 381.2)
- added D76: D_Small, Diode_SMD:D_0805_2012Metric, F.Cu at (135.5, 378.1)
- added D77: D_Small, Diode_SMD:D_0805_2012Metric, F.Cu at (131.0, 378.1)
- added D78: D_Small, Diode_SMD:D_0805_2012Metric, F.Cu at (293.8, 304.1)
- added D79: D_Small, Diode_SMD:D_0805_2012Metric, F.Cu at (314.0, 283.9)
- added D8: D_Small, Diode_SMD:D_0805_2012Metric, F.Cu at (352.3, 238.5)
- added D80: D_Small, Diode_SMD:D_0805_2012Metric, F.Cu at (318.5, 283.9)
- added D81: D_Small, Diode_SMD:D_0805_2012Metric, F.Cu at (314.0, 286.9)
- added D82: D_Small, Diode_SMD:D_0805_2012Metric, F.Cu at (298.3, 304.1)
- added D83: D_Small, Diode_SMD:D_0805_2012Metric, F.Cu at (293.8, 307.1)
- added D84: D_Small, Diode_SMD:D_0805_2012Metric, F.Cu at (352.3, 247.6)
- added D9: D_Small, Diode_SMD:D_0805_2012Metric, F.Cu at (352.3, 235.5)
- added DELETE1: MX-NoLED, MX_Only:MXOnly-1U-NoLED, F.Cu at (358.3, 98.5)
- added DOT1: MX-NoLED, MX_Only:MXOnly-1U-NoLED, F.Cu at (267.8, 174.7)
- added DOWN1: MX-NoLED, MX_Only:MXOnly-1U-NoLED, F.Cu at (339.2, 193.7)
- added D_KEY1: MX-NoLED, MX_Only:MXOnly-1U-NoLED, F.Cu at (144.0, 155.6)
- added E1: MX-NoLED, MX_Only:MXOnly-1U-NoLED, F.Cu at (139.2, 136.6)
- added EIGHT1: MX-NoLED, MX_Only:MXOnly-1U-NoLED, F.Cu at (224.9, 117.5)
- added END1: MX-NoLED, MX_Only:MXOnly-1U-NoLED, F.Cu at (358.3, 174.7)
- added ENTER1: MX-NoLED, MX_Only:MXOnly-2U-NoLED, F.Cu at (327.3, 155.6)
- added EQUAL1: MX-NoLED, MX_Only:MXOnly-1U-NoLED, F.Cu at (301.1, 117.5)
- added ESC1: MX-NoLED, MX_Only:MXOnly-1U-NoLED, F.Cu at (72.5, 98.5)
- added F1: MX-NoLED, MX_Only:MXOnly-1U-NoLED, F.Cu at (91.5, 98.5)
- added F10: MX-NoLED, MX_Only:MXOnly-1U-NoLED, F.Cu at (263.0, 98.5)
- added F11: MX-NoLED, MX_Only:MXOnly-1U-NoLED, F.Cu at (282.1, 98.5)
- added F12: MX-NoLED, MX_Only:MXOnly-1U-NoLED, F.Cu at (301.1, 98.5)
- added F2: MX-NoLED, MX_Only:MXOnly-1U-NoLED, F.Cu at (110.6, 98.5)
- added F3: MX-NoLED, MX_Only:MXOnly-1U-NoLED, F.Cu at (129.7, 98.5)
- added F4: MX-NoLED, MX_Only:MXOnly-1U-NoLED, F.Cu at (148.7, 98.5)
- added F5: MX-NoLED, MX_Only:MXOnly-1U-NoLED, F.Cu at (167.7, 98.5)
- added F6: MX-NoLED, MX_Only:MXOnly-1U-NoLED, F.Cu at (186.8, 98.5)
- added F7: MX-NoLED, MX_Only:MXOnly-1U-NoLED, F.Cu at (205.8, 98.5)
- added F8: MX-NoLED, MX_Only:MXOnly-1U-NoLED, F.Cu at (224.9, 98.5)
- added F9: MX-NoLED, MX_Only:MXOnly-1U-NoLED, F.Cu at (243.9, 98.5)
- added FIVE1: MX-NoLED, MX_Only:MXOnly-1U-NoLED, F.Cu at (167.8, 117.5)
- added FN1: MX-NoLED, MX_Only:MXOnly-1U-NoLED, F.Cu at (282.1, 193.7)
- added FOUR1: MX-NoLED, MX_Only:MXOnly-1U-NoLED, F.Cu at (148.7, 117.5)
- added F_KEY1: MX-NoLED, MX_Only:MXOnly-1U-NoLED, F.Cu at (163.0, 155.6)
- added G1: MX-NoLED, MX_Only:MXOnly-1U-NoLED, F.Cu at (182.1, 155.6)
- added H1: MX-NoLED, MX_Only:MXOnly-1U-NoLED, F.Cu at (201.1, 155.6)
- added HOME1: MX-NoLED, MX_Only:MXOnly-1U-NoLED, F.Cu at (358.2, 117.5)
- added I1: MX-NoLED, MX_Only:MXOnly-1U-NoLED, F.Cu at (234.4, 136.6)
- added INSERT1: MX-NoLED, MX_Only:MXOnly-1U-NoLED, F.Cu at (320.2, 98.5)
- added J1: MX-NoLED, MX_Only:MXOnly-1U-NoLED, F.Cu at (220.1, 155.6)
- added J2: USB_C_Receptacle_USB2.0, Connector_USB:USB_C_Receptacle_HRO_TYPE-C-31-M-12, F.Cu at (108.2, 370.9)
- added K1: MX-NoLED, MX_Only:MXOnly-1U-NoLED, F.Cu at (239.2, 155.6)
- added L1: MX-NoLED, MX_Only:MXOnly-1U-NoLED, F.Cu at (258.3, 155.6)
- added LEFT1: MX-NoLED, MX_Only:MXOnly-1U-NoLED, F.Cu at (320.1, 193.7)
- added L_ALT1: MX-NoLED, MX_Only:MXOnly-1U-NoLED, F.Cu at (122.5, 193.7)
- added L_BRACKET1: MX-NoLED, MX_Only:MXOnly-1U-NoLED, F.Cu at (291.6, 136.6)
- added L_CTRL1: MX-NoLED, MX_Only:MXOnly-1U-NoLED, F.Cu at (74.9, 193.7)
- added L_SHIFT1: MX-NoLED, MX_Only:MXOnly-2U-NoLED, F.Cu at (84.4, 174.6)
- added M1: MX-NoLED, MX_Only:MXOnly-1U-NoLED, F.Cu at (229.7, 174.7)
- added MINUS1: MX-NoLED, MX_Only:MXOnly-1U-NoLED, F.Cu at (282.1, 117.5)
- added N1: MX-NoLED, MX_Only:MXOnly-1U-NoLED, F.Cu at (210.6, 174.7)
- added NINE1: MX-NoLED, MX_Only:MXOnly-1U-NoLED, F.Cu at (243.9, 117.5)
- added O1: MX-NoLED, MX_Only:MXOnly-1U-NoLED, F.Cu at (253.5, 136.6)
- added ONE1: MX-NoLED, MX_Only:MXOnly-1U-NoLED, F.Cu at (91.5, 117.5)
- added P1: MX-NoLED, MX_Only:MXOnly-1U-NoLED, F.Cu at (272.5, 136.6)
- added PRTSC1: MX-NoLED, MX_Only:MXOnly-1U-NoLED, F.Cu at (339.2, 98.5)
- added Q1: MX-NoLED, MX_Only:MXOnly-1U-NoLED, F.Cu at (101.1, 136.6)
- added R1: 22, Resistor_SMD:R_0815_2038Metric, F.Cu at (216.3, 276.9)
- added R10: 5.1k, Resistor_SMD:R_0815_2038Metric, F.Cu at (220.7, 265.6)
- added R11: 5.1k, Resistor_SMD:R_0815_2038Metric, F.Cu at (216.3, 265.6)
- added R2: 22, Resistor_SMD:R_0815_2038Metric, F.Cu at (211.8, 276.9)
- added R3: 10k, Resistor_SMD:R_0815_2038Metric, F.Cu at (220.7, 271.2)
- added R5: 10k, Resistor_SMD:R_0815_2038Metric, F.Cu at (211.8, 265.6)
- added R6: 10k, Resistor_SMD:R_0815_2038Metric, F.Cu at (116.3, 367.3)
- added R7: 10k, Resistor_SMD:R_0815_2038Metric, F.Cu at (216.3, 271.2)
- added R8: 10k, Resistor_SMD:R_0815_2038Metric, F.Cu at (211.8, 271.2)
- added R9: 10k, Resistor_SMD:R_0815_2038Metric, F.Cu at (225.2, 265.6)
- added RIGHT1: MX-NoLED, MX_Only:MXOnly-1U-NoLED, F.Cu at (358.2, 193.7)
- added R_ALT1: MX-NoLED, MX_Only:MXOnly-1U-NoLED, F.Cu at (263.0, 193.7)
- added R_BRACKET1: MX-NoLED, MX_Only:MXOnly-1U-NoLED, F.Cu at (310.6, 136.6)
- added R_CTRL1: MX-NoLED, MX_Only:MXOnly-1U-NoLED, F.Cu at (301.1, 193.7)
- added R_KEY1: MX-NoLED, MX_Only:MXOnly-1U-NoLED, F.Cu at (158.2, 136.6)
- added R_SHIFT1: MX-NoLED, MX_Only:MXOnly-1U-NoLED, F.Cu at (313.0, 174.7)
- added S1: MX-NoLED, MX_Only:MXOnly-1U-NoLED, F.Cu at (124.9, 155.6)
- added SEMICOLON1: MX-NoLED, MX_Only:MXOnly-1U-NoLED, F.Cu at (277.3, 155.6)
- added SEVEN1: MX-NoLED, MX_Only:MXOnly-1U-NoLED, F.Cu at (205.9, 117.5)
- added SIX1: MX-NoLED, MX_Only:MXOnly-1U-NoLED, F.Cu at (186.8, 117.5)
- added SLASH1: MX-NoLED, MX_Only:MXOnly-1U-NoLED, F.Cu at (286.8, 174.7)
- added SPACE1: MX-NoLED, MX_Only:MXOnly-6.25U-ReversedStabilizers-NoLED, F.Cu at (194.0, 193.7)
- added SW1: SW_Push, Keebio-Parts:SW_SPST_3x3, F.Cu at (72.1, 382.5)
- added SW2: Rotary_Encoder_Switch, Keebio-Parts:RotaryEncoder_EC11, F.Cu at (358.2, 146.2)
- added T1: MX-NoLED, MX_Only:MXOnly-1U-NoLED, F.Cu at (177.3, 136.6)
- added TAB1: MX-NoLED, MX_Only:MXOnly-1U-NoLED, F.Cu at (77.3, 136.6)
- added THREE1: MX-NoLED, MX_Only:MXOnly-1U-NoLED, F.Cu at (129.7, 117.5)
- added TWO1: MX-NoLED, MX_Only:MXOnly-1U-NoLED, F.Cu at (110.6, 117.5)
- added U1: ATmega32U4-AU, Package_QFP:TQFP-44_10x10mm_P0.8mm, F.Cu at (95.1, 372.3)
- added UP1: MX-NoLED, MX_Only:MXOnly-1U-NoLED, F.Cu at (339.2, 174.6)
- added U_KEY1: MX-NoLED, MX_Only:MXOnly-1U-NoLED, F.Cu at (215.4, 136.6)
- added V1: MX-NoLED, MX_Only:MXOnly-1U-NoLED, F.Cu at (172.5, 174.7)
- added W1: MX-NoLED, MX_Only:MXOnly-1U-NoLED, F.Cu at (120.1, 136.6)
- added WIN1: MX-NoLED, MX_Only:MXOnly-1U-NoLED, F.Cu at (98.7, 193.7)
- added X1: MX-NoLED, MX_Only:MXOnly-1U-NoLED, F.Cu at (134.5, 174.7)
- added Y1: 16MHz, Crystal:Crystal_SMD_3225-4Pin_3.2x2.5mm, F.Cu at (90.5, 381.8)
- added Y_KEY1: MX-NoLED, MX_Only:MXOnly-1U-NoLED, F.Cu at (196.3, 136.6)
- added Z1: MX-NoLED, MX_Only:MXOnly-1U-NoLED, F.Cu at (115.4, 174.7)
- added ZERO1: MX-NoLED, MX_Only:MXOnly-1U-NoLED, F.Cu at (263.0, 117.5)

Commit message: Placing diodes to the corresponding swtiches
Parts:
- D1, D10, D11, D12, D13, D14, D15, D16, D17, D18, D19, D2, D20, D21, D22, D23, D24, D25, D27, D28, D29, D3, D30, D31, D32, D33, D34, D35, D36, D37, D38, D39, D4, D40, D41, D42, D43, D44, D45, D46, D47, D48, D49, D5, D50, D51, D52, D53, D54, D55, D56, D57, D58, D59, D6, D60, D61, D62, D63, D64, D65, D66, D67, D68, D69, D7, D70, D71, D72, D73, D74, D75, D76, D77, D78, D79, D8, D80, D81, D82, D83, D84, D9: moved to B.Cu
- moved D75 367.3 mm to (348.8, 95.7), turned to 90 degrees
- moved D70 357.8 mm to (329.7, 95.7), turned to 90 degrees
- moved D65 336.7 mm to (310.6, 95.7), turned to 90 degrees
- moved D59 335.8 mm to (291.6, 95.7), turned to 90 degrees
- moved D71 334.2 mm to (320.1, 133.7), turned to 90 degrees
- moved D76 331.9 mm to (337.3, 114.7), turned to 90 degrees
- moved D67 331.4 mm to (301.1, 133.7), turned to 90 degrees
- moved D54 331.1 mm to (272.6, 114.7), turned to 90 degrees
- moved D53 328.2 mm to (272.6, 95.7), turned to 90 degrees
- moved D77 324.2 mm to (344.0, 133.7), turned to 90 degrees
- moved D60 312.8 mm to (291.6, 114.7), turned to 90 degrees
- moved D68 307.6 mm to (305.9, 152.7), turned to 90 degrees
- moved D1 303.5 mm to (82.0, 95.7), turned to 90 degrees
- moved D43 302.4 mm to (234.4, 95.7), turned to 90 degrees
- moved D72 299.5 mm to (334.9, 152.7), turned to 90 degrees
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Routing:
- net Net-(D10-Pad2): track 0.00 -> 7.59 mm
- net Net-(D1-Pad2): track 0.00 -> 7.55 mm
- net Net-(D6-Pad2): track 0.00 -> 7.54 mm
- net Net-(BACKTICK1-Pad2): track 0.00 -> 7.50 mm
- net Net-(CAPSLOCK1-Pad2): track 0.00 -> 7.48 mm

Commit message: Connecting switch matrix
Parts:
- added C7: 10uF, Capacitor_SMD:C_0805_2012Metric, B.Cu at (225.2, 195.9)
- C1, C10, C2, C3, C4, C5, C6, C8, C9, J2, SW1, U1, Y1: moved to B.Cu
- R1, R10, R11, R2, R3, R5, R6, R7, R8, R9: footprint Resistor_SMD:R_0815_2038Metric -> Keebio-Parts:R_0805; moved to B.Cu
- moved J2 370.2 mm to (348.7, 89.4)
- moved R11 235.9 mm to (364.0, 81.7), turned to 90 degrees
- moved Y1 231.0 mm to (233.5, 200.3)
- moved U1 227.8 mm to (233.2, 191.2), turned to 180 degrees
- moved R10 225.0 mm to (346.2, 78.8), turned to 90 degrees
- moved SW1 149.9 mm to (184.7, 283.6)
- moved C3 144.8 mm to (238.2, 200.3), turned to 90 degrees
- moved C6 141.3 mm to (226.8, 184.7), turned to 135 degrees
- moved C1 133.8 mm to (239.9, 184.6), turned to 45 degrees
- moved C2 133.0 mm to (229.0, 200.3), turned to 270 degrees
- moved R6 127.0 mm to (199.1, 270.9)
- moved C4 105.9 mm to (243.7, 222.0), turned to 180 degrees
- moved C5 102.3 mm to (251.1, 221.0)
- moved C8 95.6 mm to (227.3, 293.0), turned to 180 degrees
- moved R5 39.3 mm to (245.6, 285.8), turned to 90 degrees
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Connections:
- C10 pad 2: Net-(C10-Pad2) -> EC11A_M
- C9 pad 1: Net-(C9-Pad1) -> EC11B_M
- R6 pad 2: Net-(C9-Pad1) -> EC11B_M
- R7 pad 2: Net-(C10-Pad2) -> EC11A_M
- U1 pad 26: Net-(C9-Pad1) -> Net-(U1-Pad26)
- U1 pad 27: Net-(C10-Pad2) -> Net-(U1-Pad27)
Routing:
- net ROW1: track 0.00 -> 285.6 mm
- net ROW0: track 0.06 -> 285.4 mm
- net ROW3: track 0.00 -> 280.4 mm
- net ROW2: track 0.00 -> 257.2 mm
- net COL13: track 0.00 -> 122.0 mm
- net COL3: track 0.00 -> 110.1 mm
- net COL1: track 0.00 -> 107.8 mm
- net COL10: track 0.00 -> 107.1 mm
- net COL11: track 0.00 -> 107.1 mm
- net COL6: track 0.00 -> 106.1 mm
- net COL12: track 0.00 -> 104.9 mm
- net COL14: track 0.00 -> 103.1 mm
- net COL0: track 0.00 -> 102.1 mm
- net COL15: track 0.00 -> 96.4 mm
- net COL2: track 0.00 -> 86.1 mm
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Other:
- net class Power added: clearance 0.2, trace_width 0.381, via_dia 0.8, via_drill 0.4

Commit message: Connecting the rest
Parts:
- C1, C10, C2, C3, C4, C5, C6, C7, C8, C9: footprint Capacitor_SMD:C_0805_2012Metric -> Capacitor_SMD:C_0603_1608Metric
- R1, R10, R11, R2, R3, R5, R6, R7, R8, R9: footprint Keebio-Parts:R_0805 -> Keebio-Parts:R_0603
- moved R1 227.4 mm to (349.4, 99.0), turned to 90 degrees
- moved R2 224.7 mm to (348.0, 99.0), turned to 90 degrees
- moved R6 195.9 mm to (360.8, 160.4), turned to 270 degrees
- moved R8 187.7 mm to (360.1, 156.2), turned to 180 degrees
- moved R7 178.1 mm to (355.9, 160.6), turned to 270 degrees
- moved R9 169.8 mm to (355.0, 156.2), turned to 180 degrees
- moved C9 146.1 mm to (361.6, 158.4)
- moved C10 134.1 mm to (356.7, 158.4), turned to 180 degrees
- moved SW1 112.5 mm to (248.5, 190.9), turned to 90 degrees
- moved C8 103.7 mm to (245.1, 190.8), turned to 0 degrees
- moved R5 102.1 mm to (224.1, 186.0), turned to 315 degrees
- moved R3 78.3 mm to (245.3, 196.9), turned to 225 degrees
- moved C4 33.2 mm to (245.1, 188.8), turned to 0 degrees
- moved C5 28.8 mm to (245.1, 192.8)
- moved R11 21.7 mm to (350.9, 99.0)
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Connections:
- net Net-(R1-Pad1) renamed D_P
- net Net-(R2-Pad1) renamed D_N
- U1 pad 10: Net-(U1-Pad10) -> COL2
- U1 pad 11: Net-(U1-Pad11) -> COL3
- U1 pad 12: Net-(U1-Pad12) -> COL4
- U1 pad 18: Net-(U1-Pad18) -> COL5
- U1 pad 19: Net-(U1-Pad19) -> COL6
- U1 pad 20: Net-(U1-Pad20) -> ROW5
- U1 pad 21: Net-(U1-Pad21) -> ROW4
- U1 pad 22: Net-(U1-Pad22) -> ROW3
- U1 pad 25: Net-(U1-Pad25) -> ROW0
- U1 pad 26: Net-(U1-Pad26) -> ROW1
- U1 pad 27: Net-(U1-Pad27) -> ROW2
- U1 pad 28: Net-(U1-Pad28) -> COL7
- U1 pad 29: Net-(U1-Pad29) -> COL8
- U1 pad 30: Net-(U1-Pad30) -> COL9
- U1 pad 31: Net-(U1-Pad31) -> COL10
- U1 pad 32: Net-(U1-Pad32) -> COL15
- U1 pad 36: Net-(U1-Pad36) -> EC11A_M
- U1 pad 37: Net-(U1-Pad37) -> EC11B_M
- U1 pad 38: Net-(U1-Pad38) -> COL14
- U1 pad 39: Net-(U1-Pad39) -> COL13
- U1 pad 40: Net-(U1-Pad40) -> COL12
- U1 pad 41: Net-(U1-Pad41) -> COL11
- U1 pad 8: Net-(U1-Pad8) -> COL0
- U1 pad 9: Net-(U1-Pad9) -> COL1
Routing:
- net ROW5: track 0.00 -> 349.5 mm, vias 0 -> 2
- net GND: track 80.1 -> 422.5 mm, vias 0 -> 4
- net ROW4: track 0.00 -> 324.4 mm, vias 0 -> 2
- net +5V: track 6.52 -> 323.0 mm, vias 0 -> 9
- net ROW0: track 285.4 -> 573.4 mm
- net COL11: track 107.1 -> 375.6 mm
- net ROW1: track 285.6 -> 553.0 mm
- net ROW2: track 257.2 -> 508.9 mm
- net COL12: track 104.9 -> 353.7 mm
- net COL13: track 122.0 -> 350.9 mm
- net D_P: track 0.00 -> 220.8 mm, vias 0 -> 2
- net D_N: track 0.00 -> 220.4 mm, vias 0 -> 2
- net COL14: track 103.1 -> 312.3 mm
- net COL15: track 96.4 -> 302.1 mm
- net COL0: track 102.1 -> 301.8 mm, vias 0 -> 1
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
Commit message: Fixing some track to close too pad
Parts:
- moved SPACE1 0.05 mm to (193.9, 193.7)
Routing:
- net GND: track 422.5 -> 400.8 mm, vias 4 -> 1
- net ROW3: track 352.1 -> 351.5 mm
- net ROW4: track 324.4 -> 323.8 mm

Commit message: Editing B.SilkS layer
Routing:
- net GND: track 400.8 -> 389.6 mm
